File: devel/devel/Button_PU.sch (KiCad schematic (older format))
At the start: 3 parts, among them SW1 SW

Commit message: Completed the PCB desing for devel, ready to etch
Changed lines of the file:
@@
 AR Path="/5C594511/5C58179F" Ref="R14"  Part="1"
 AR Path="/5C5956B5/5C58179F" Ref="R23"  Part="1"
-F 0 "R12" H 3470 2296 50  0000 L CNN
+F 0 "R4" H 3470 2296 50  0000 L CNN
 F 1 "10k" H 3470 2205 50  0000 L CNN
 F 2 "Resistor_SMD:R_0805_2012Metric_Pad1.15x1.40mm_HandSolder" V 3330 2250 50  0001 C CNN
@@
 AR Path="/5C594511/5C581B3D" Ref="SW14"  Part="1"
 AR Path="/5C5956B5/5C581B3D" Ref="SW15"  Part="1"
-F 0 "SW12" V 3354 2748 50  0000 L CNN
+F 0 "SW4" V 3354 2748 50  0000 L CNN
 F 1 "SW" V 3445 2748 50  0000 L CNN
 F 2 "Button_Switch_SMD:SW_SPST_EVQQ2" H 3400 2800 50  0001 C CNN
@@
 AR Path="/5C594511/5C581BEA" Ref="C15"  Part="1"
 AR Path="/5C5956B5/5C581BEA" Ref="C16"  Part="1"
-F 0 "C12" H 4115 2646 50  0000 L CNN
+F 0 "C4" H 4115 2646 50  0000 L CNN
 F 1 "10n" H 4115 2555 50  0000 L CNN
 F 2 "Capacitor_SMD:C_0805_2012Metric_Pad1.15x1.40mm_HandSolder" H 4038 2450 50  0001 C CNN
