File: devel/devel/devel.kicad_pcb (KiCad board)
At the start: 2 copper layers, 7 parts, among them SW1 SW_Push, SW2 SW_Push

Commit message: Worked on the dev-board
Parts:
- added C10: 10n, Capacitor_SMD:C_0805_2012Metric_Pad1.15x1.40mm_HandSolder, F.Cu at (233.0, 89.7)
- added C11: 10n, Capacitor_SMD:C_0805_2012Metric_Pad1.15x1.40mm_HandSolder, F.Cu at (178.6, 96.2)
- added C12: 10n, Capacitor_SMD:C_0805_2012Metric_Pad1.15x1.40mm_HandSolder, F.Cu at (277.6, 92.7)
- added C13: C, Capacitor_SMD:C_0805_2012Metric_Pad1.15x1.40mm_HandSolder, F.Cu at (15.4, 106.2)
- added C14: 10n, Capacitor_SMD:C_0805_2012Metric_Pad1.15x1.40mm_HandSolder, F.Cu at (232.9, 126.2)
- added C15: 10n, Capacitor_SMD:C_0805_2012Metric_Pad1.15x1.40mm_HandSolder, F.Cu at (215.6, 126.5)
- added C16: 10n, Capacitor_SMD:C_0805_2012Metric_Pad1.15x1.40mm_HandSolder, F.Cu at (171.8, 133.9)
- added C3: 10n, Capacitor_SMD:C_0805_2012Metric_Pad1.15x1.40mm_HandSolder, F.Cu at (185.3, 110.4)
- added C4: 10n, Capacitor_SMD:C_0805_2012Metric_Pad1.15x1.40mm_HandSolder, F.Cu at (210.9, 107.7)
- added C5: 10n, Capacitor_SMD:C_0805_2012Metric_Pad1.15x1.40mm_HandSolder, F.Cu at (250.2, 97.1)
- added C6: 10n, Capacitor_SMD:C_0805_2012Metric_Pad1.15x1.40mm_HandSolder, F.Cu at (236.8, 108.6)
- added C7: 10n, Capacitor_SMD:C_0805_2012Metric_Pad1.15x1.40mm_HandSolder, F.Cu at (261.2, 107.3)
- added C8: 10n, Capacitor_SMD:C_0805_2012Metric_Pad1.15x1.40mm_HandSolder, F.Cu at (250.7, 119.4)
- added C9: 10n, Capacitor_SMD:C_0805_2012Metric_Pad1.15x1.40mm_HandSolder, F.Cu at (216.2, 88.1)
- added D1: LED, LED_SMD:LED_0603_1608Metric_Pad1.05x0.95mm_HandSolder, F.Cu at (120.6, 25.0)
- added D2: LED, LED_SMD:LED_0603_1608Metric_Pad1.05x0.95mm_HandSolder, F.Cu at (118.2, 25.0)
- added D3: LED, LED_SMD:LED_0603_1608Metric_Pad1.05x0.95mm_HandSolder, F.Cu at (115.6, 25.1)
- added D4: LED, LED_SMD:LED_0603_1608Metric_Pad1.05x0.95mm_HandSolder, F.Cu at (113.0, 25.1)
- added D5: LED, LED_SMD:LED_0603_1608Metric_Pad1.05x0.95mm_HandSolder, F.Cu at (110.4, 24.9)
- added D6: LED, LED_SMD:LED_0603_1608Metric_Pad1.05x0.95mm_HandSolder, F.Cu at (107.8, 24.8)
- added D7: LED, LED_SMD:LED_0603_1608Metric_Pad1.05x0.95mm_HandSolder, F.Cu at (105.4, 24.7)
- added D8: LED, LED_SMD:LED_0603_1608Metric_Pad1.05x0.95mm_HandSolder, F.Cu at (102.8, 24.7)
- added R10: 10k, Resistor_SMD:R_0805_2012Metric_Pad1.15x1.40mm_HandSolder, F.Cu at (233.0, 87.7)
- added R11: 10k, Resistor_SMD:R_0805_2012Metric_Pad1.15x1.40mm_HandSolder, F.Cu at (178.6, 94.3)
- added R12: 10k, Resistor_SMD:R_0805_2012Metric_Pad1.15x1.40mm_HandSolder, F.Cu at (277.6, 94.6)
- added R13: 10k, Resistor_SMD:R_0805_2012Metric_Pad1.15x1.40mm_HandSolder, F.Cu at (232.9, 124.2)
- added R14: 10k, Resistor_SMD:R_0805_2012Metric_Pad1.15x1.40mm_HandSolder, F.Cu at (215.6, 124.6)
- added R15: R, Resistor_SMD:R_0805_2012Metric_Pad1.15x1.40mm_HandSolder, F.Cu at (120.6, 19.8)
- added R16: R, Resistor_SMD:R_0805_2012Metric_Pad1.15x1.40mm_HandSolder, F.Cu at (118.2, 19.8)
- added R17: R, Resistor_SMD:R_0805_2012Metric_Pad1.15x1.40mm_HandSolder, F.Cu at (115.6, 19.8)
- added R18: R, Resistor_SMD:R_0805_2012Metric_Pad1.15x1.40mm_HandSolder, F.Cu at (113.0, 19.7)
- added R19: R, Resistor_SMD:R_0805_2012Metric_Pad1.15x1.40mm_HandSolder, F.Cu at (110.4, 19.6)
- added R20: R, Resistor_SMD:R_0805_2012Metric_Pad1.15x1.40mm_HandSolder, F.Cu at (107.9, 19.8)
- added R21: R, Resistor_SMD:R_0805_2012Metric_Pad1.15x1.40mm_HandSolder, F.Cu at (105.4, 19.8)
- added R22: R, Resistor_SMD:R_0805_2012Metric_Pad1.15x1.40mm_HandSolder, F.Cu at (102.8, 19.8)
- added R23: 10k, Resistor_SMD:R_0805_2012Metric_Pad1.15x1.40mm_HandSolder, F.Cu at (171.8, 135.8)
- added R3: 10k, Resistor_SMD:R_0805_2012Metric_Pad1.15x1.40mm_HandSolder, F.Cu at (185.3, 108.4)
- added R4: 10k, Resistor_SMD:R_0805_2012Metric_Pad1.15x1.40mm_HandSolder, F.Cu at (210.9, 109.6)
- added R5: 10k, Resistor_SMD:R_0805_2012Metric_Pad1.15x1.40mm_HandSolder, F.Cu at (250.2, 99.1)
- added R6: 10k, Resistor_SMD:R_0805_2012Metric_Pad1.15x1.40mm_HandSolder, F.Cu at (236.8, 106.6)
- added R7: 10k, Resistor_SMD:R_0805_2012Metric_Pad1.15x1.40mm_HandSolder, F.Cu at (261.2, 105.4)
- added R8: 10k, Resistor_SMD:R_0805_2012Metric_Pad1.15x1.40mm_HandSolder, F.Cu at (250.7, 117.5)
- added R9: 10k, Resistor_SMD:R_0805_2012Metric_Pad1.15x1.40mm_HandSolder, F.Cu at (216.2, 90.0)
- added RV1: R_POT, Potentiometer_THT:Potentiometer_Alps_RK163_Single_Horizontal, F.Cu at (41.4, 110.0)
- added SW10: SW, Button_Switch_SMD:SW_SPST_EVQQ2, F.Cu at (225.9, 90.0)
- added SW11: SW, Button_Switch_SMD:SW_SPST_EVQQ2, F.Cu at (171.5, 96.6)
- added SW12: SW, Button_Switch_SMD:SW_SPST_EVQQ2, F.Cu at (270.5, 95.0)
- added SW13: SW, Button_Switch_SMD:SW_SPST_EVQQ2, F.Cu at (225.8, 126.5)
- added SW14: SW, Button_Switch_SMD:SW_SPST_EVQQ2, F.Cu at (208.5, 126.9)
- added SW15: SW, Button_Switch_SMD:SW_SPST_EVQQ2, F.Cu at (164.7, 136.2)
- added SW3: SW, Button_Switch_SMD:SW_SPST_EVQQ2, F.Cu at (178.1, 110.7)
- added SW4: SW, Button_Switch_SMD:SW_SPST_EVQQ2, F.Cu at (203.8, 110.0)
- added SW5: SW, Button_Switch_SMD:SW_SPST_EVQQ2, F.Cu at (243.1, 99.4)
- added SW6: SW, Button_Switch_SMD:SW_SPST_EVQQ2, F.Cu at (229.6, 108.9)
- added SW7: SW, Button_Switch_SMD:SW_SPST_EVQQ2, F.Cu at (254.0, 107.7)
- added SW8: SW, Button_Switch_SMD:SW_SPST_EVQQ2, F.Cu at (243.6, 119.8)
- added SW9: SW, Button_Switch_SMD:SW_SPST_EVQQ2, F.Cu at (209.0, 90.4)
- C1, C2: footprint Capacitor_SMD:C_0603_1608Metric -> Capacitor_SMD:C_0805_2012Metric_Pad1.15x1.40mm_HandSolder
- R1, R2: footprint Resistor_SMD:R_0603_1608Metric -> Resistor_SMD:R_0805_2012Metric_Pad1.15x1.40mm_HandSolder
- SW1, SW2: value SW_Push -> SW
- moved SW1 148.9 mm to (190.3, 103.2), turned to 0 degrees
- moved SW2 147.1 mm to (190.9, 116.8)
- moved C1 146.8 mm to (197.4, 100.9)
- moved R1 146.6 mm to (197.4, 102.8), turned to 0 degrees
- moved C2 145.9 mm to (198.1, 116.5), turned to 0 degrees
- moved R2 143.2 mm to (198.1, 114.5), turned to 0 degrees
- moved A1 23.7 mm to (85.6, 86.0)
Connections:
- A1 pad 10: (no net) -> /P0.04
- A1 pad 11: (no net) -> /P0.28
- A1 pad 12: (no net) -> /P0.29
- A1 pad 13: (no net) -> /P0.30
- A1 pad 14: (no net) -> /P0.31
- A1 pad 15: (no net) -> /P0.11
- A1 pad 16: (no net) -> /P0.12
- A1 pad 17: (no net) -> /P0.13
- A1 pad 18: (no net) -> /P0.14
- A1 pad 19: (no net) -> /P0.15
- A1 pad 2: /VDD -> (no net)
- A1 pad 20: (no net) -> /P0.16
- A1 pad 22: (no net) -> /P0.18
- A1 pad 23: (no net) -> /P0.19
- A1 pad 24: (no net) -> /P0.20
- A1 pad 26: (no net) -> /P0.23
- A1 pad 27: (no net) -> /P0.24
- A1 pad 28: (no net) -> /P0.25
- A1 pad 3: (no net) -> /RESET
- A1 pad 30: (no net) -> /P0.02
- A1 pad 31: (no net) -> /P0.26
- A1 pad 32: (no net) -> /P0.27
- A1 pad 9: (no net) -> /P0.03(A0)
- C1 pad 1: /P0.17 -> /P0.19
- C2 pad 1: /P0.22 -> /P0.20
- R1 pad 2: /P0.17 -> /P0.19
- R2 pad 2: /P0.22 -> /P0.20
- SW1 pad 1: /P0.17 -> /P0.19
- SW2 pad 1: /P0.22 -> /P0.20
Routing:
- net /VDD: track 50.9 -> 0.00 mm
- net /GND: track 57.6 -> 14.0 mm
- net /5V: track 37.8 -> 0.00 mm
- net /P0.22: track 13.2 -> 0.00 mm
- net /P0.17: track 7.37 -> 0.06 mm
- net Net-(D4-Pad2): track 0.00 -> 3.50 mm
- net Net-(D5-Pad2): track 0.00 -> 3.43 mm
- net Net-(D3-Pad2): track 0.00 -> 3.38 mm
- net Net-(D2-Pad2): track 0.00 -> 3.31 mm
- net Net-(D1-Pad2): track 0.00 -> 3.30 mm
- net Net-(D6-Pad2): track 0.00 -> 3.10 mm
- net Net-(D8-Pad2): track 0.00 -> 2.95 mm
- net Net-(D7-Pad2): track 0.00 -> 2.95 mm
Other:
- net class Default: clearance 0.2 -> 0.45; trace_width 0.25 -> 0.8; via_dia 0.8 -> 3; via_drill 0.4 -> 1.6
- rule trace_clearance: 0.2 -> 0.45

Commit message: Make a physical border
Parts:
- moved C13 55.2 mm to (27.8, 159.9)
- moved RV1 53.8 mm to (40.4, 163.8)
- moved C12 45.6 mm to (236.6, 112.7)
- moved C7 45.6 mm to (220.2, 127.3)
- moved R12 45.6 mm to (236.6, 114.6)
- moved R7 45.6 mm to (220.2, 125.4)
- moved C1 45.6 mm to (156.4, 120.9)
- moved C10 45.6 mm to (192.0, 109.7)
- moved C11 45.6 mm to (137.6, 116.2)
- moved C15 45.6 mm to (174.6, 146.5)
- moved C16 45.6 mm to (130.8, 153.9)
- moved C2 45.6 mm to (157.1, 136.5)
- moved C4 45.6 mm to (169.9, 127.7)
- moved C5 45.6 mm to (209.2, 117.1)
- moved C8 45.6 mm to (209.7, 139.4)
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Routing:
- net /GND: track 14.0 -> 12.9 mm

Commit message: Completed the PCB desing for devel, ready to etch
Parts:
- moved R12 146.0 mm to (109.8, 42.2)
- moved R7 136.7 mm to (109.7, 44.8)
- moved R4 135.0 mm to (52.5, 63.0), turned to 270 degrees
- moved R8 131.2 mm to (110.0, 52.2)
- moved C12 130.4 mm to (125.5, 44.5), turned to 270 degrees
- moved RV1 128.2 mm to (91.0, 46.0), turned to 90 degrees
- moved SW15 124.6 mm to (65.5, 46.0)
- moved R23 124.1 mm to (75.0, 45.0), turned to 90 degrees
- moved C16 123.5 mm to (72.5, 45.0), turned to 270 degrees
- moved SW4 123.1 mm to (58.9, 64.0), turned to 180 degrees
- moved R5 122.7 mm to (109.8, 47.2)
- moved R3 120.5 mm to (51.5, 51.5), turned to 180 degrees
- moved SW12 119.5 mm to (132.9, 44.5)
- moved C15 118.8 mm to (73.0, 85.0), turned to 90 degrees
- moved SW2 117.9 mm to (52.1, 71.0), turned to 180 degrees
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Connections:
- A1 pad 5: /5V -> (no net)
- C1 pad 1: /P0.19 -> /P0.28
- C10 pad 1: /P0.30 -> /P0.22
- C11 pad 1: /P0.25 -> /P0.31
- C12 pad 1: /P0.31 -> /P0.27
- C14 pad 1: /P0.26 -> /P0.12
- C15 pad 1: /P0.27 -> /P0.11
- C2 pad 1: /P0.20 -> /P0.29
- C3 pad 1: /P0.22 -> /P0.30
- C4 pad 1: /P0.23 -> /P0.04
- C6 pad 1: /P0.04 -> /P0.24
- C7 pad 1: /P0.28 -> /P0.26
- C8 pad 1: /P0.29 -> /P0.25
- C9 pad 1: /P0.24 -> /P0.23
- R1 pad 1: /5V -> /VDD
- R1 pad 2: /P0.19 -> /P0.28
- R10 pad 2: /P0.30 -> /P0.22
- R11 pad 1: /5V -> /VDD
- R11 pad 2: /P0.25 -> /P0.31
- R12 pad 2: /P0.31 -> /P0.27
- R13 pad 1: /5V -> /VDD
- R13 pad 2: /P0.26 -> /P0.12
- R14 pad 2: /P0.27 -> /P0.11
- R15 pad 1: /P0.11 -> /P0.13
- R16 pad 1: /P0.12 -> /P0.14
- R17 pad 1: /P0.13 -> /P0.15
- R18 pad 1: /P0.14 -> /P0.16
- R19 pad 1: /P0.15 -> /P0.17
- R2 pad 2: /P0.20 -> /P0.29
- R20 pad 1: /P0.16 -> /P0.18
- R21 pad 1: /P0.17 -> /P0.19
- R22 pad 1: /P0.18 -> /P0.20
- R3 pad 1: /5V -> /VDD
- R3 pad 2: /P0.22 -> /P0.30
- R4 pad 2: /P0.23 -> /P0.04
- R5 pad 1: /5V -> /VDD
- R6 pad 2: /P0.04 -> /P0.24
- R7 pad 1: /5V -> /VDD
- R7 pad 2: /P0.28 -> /P0.26
- R8 pad 2: /P0.29 -> /P0.25
- R9 pad 1: /5V -> /VDD
- R9 pad 2: /P0.24 -> /P0.23
- SW1 pad 1: /P0.19 -> /P0.28
- SW10 pad 1: /P0.30 -> /P0.22
- SW11 pad 1: /P0.25 -> /P0.31
- SW12 pad 1: /P0.31 -> /P0.27
- SW13 pad 1: /P0.26 -> /P0.12
- SW14 pad 1: /P0.27 -> /P0.11
- SW2 pad 1: /P0.20 -> /P0.29
- SW3 pad 1: /P0.22 -> /P0.30
- SW4 pad 1: /P0.23 -> /P0.04
- SW6 pad 1: /P0.04 -> /P0.24
- SW7 pad 1: /P0.28 -> /P0.26
- SW8 pad 1: /P0.29 -> /P0.25
- SW9 pad 1: /P0.24 -> /P0.23
Routing:
- net /GND: track 12.9 -> 385.9 mm, vias 0 -> 30
- net /VDD: track 0.00 -> 187.5 mm
- net /P0.31: track 0.00 -> 73.7 mm, vias 0 -> 2
- net /P0.30: track 0.00 -> 59.4 mm, vias 0 -> 2
- net /P0.23: track 0.00 -> 47.3 mm, vias 0 -> 2
- net /P0.11: track 0.00 -> 44.2 mm, vias 0 -> 2
- net /P0.26: track 0.00 -> 43.8 mm, vias 0 -> 2
- net /P0.28: track 0.00 -> 41.9 mm, vias 0 -> 2
- net /P0.25: track 0.00 -> 40.2 mm, vias 0 -> 2
- net /P0.13: track 0.11 -> 39.8 mm
- net /P0.03(A0): track 0.00 -> 38.6 mm
- net /P0.14: track 0.06 -> 35.5 mm
- net /P0.15: track 0.06 -> 31.5 mm
- net /P0.24: track 0.00 -> 28.7 mm, vias 0 -> 2
- net /RESET: track 0.00 -> 28.2 mm, vias 0 -> 2
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- added copper zone on F.Cu, net /GND
Other:
- net class Default: via_dia 3 -> 0.4; via_drill 1.6 -> 0.3
