File: rev-1/rev1/LED.sch (KiCad schematic (older format))
At the start: 4 parts

Commit message: More Work, almost done with rev 1
Parts:
- R1: value R -> 100R
- R2, R3: value R -> 10R
Changed lines of the file:
@@
 P 2900 3350
 F 0 "R1" H 2970 3396 50  0000 L CNN
-F 1 "R" H 2970 3305 50  0000 L CNN
+F 1 "100R" H 2970 3305 50  0000 L CNN
 F 2 "Resistor_SMD:R_0603_1608Metric" V 2830 3350 50  0001 C CNN
 F 3 "~" H 2900 3350 50  0001 C CNN
@@
 P 3100 3350
 F 0 "R2" H 3170 3396 50  0000 L CNN
-F 1 "R" H 3170 3305 50  0000 L CNN
+F 1 "10R" H 3170 3305 50  0000 L CNN
 F 2 "Resistor_SMD:R_0603_1608Metric" V 3030 3350 50  0001 C CNN
 F 3 "~" H 3100 3350 50  0001 C CNN
@@
 P 3300 3350
 F 0 "R3" H 3370 3396 50  0000 L CNN
-F 1 "R" H 3370 3305 50  0000 L CNN
+F 1 "10R" H 3370 3305 50  0000 L CNN
 F 2 "Resistor_SMD:R_0603_1608Metric" V 3230 3350 50  0001 C CNN
 F 3 "~" H 3300 3350 50  0001 C CNN
