File: rev-1/rev1/rev1.sch (KiCad schematic (older format))
At the start: 16 parts, among them J1 Conn_01x08_Female, U1 nRF52810-QFxx, X1 32MHz

Commit message: More Work, almost done with rev 1
Connections:
- net BTN_A: now also U1.41 (P0.29/AIN5); no longer U1.38 (P0.26)
- net BTN_B: now also U1.40 (P0.28/AIN4); no longer U1.37 (P0.25)
- net BTN_R: now also U1.43 (P0.31/AIN7); no longer U1.40 (P0.28/AIN4)
- net BTN_SELECT: now also U1.37 (P0.25); no longer U1.43 (P0.31/AIN7)
- net BTN_START: now also U1.38 (P0.26); no longer U1.42 (P0.30/AIN6)
- net BTN_X: now also U1.42 (P0.30/AIN6); no longer U1.39 (P0.27)
- net BTN_Y: now also U1.39 (P0.27); no longer U1.41 (P0.29/AIN5)
- net DPAD_DOWN: now also U1.19 (P0.16); no longer U1.20 (P0.17)
- net DPAD_LEFT: now also U1.18 (P0.15); no longer U1.19 (P0.16)
- net DPAD_RIGHT: now also U1.20 (P0.17); no longer U1.18 (P0.15)
Changed lines of the file:
@@
 Text Label 3800 3750 0    50   ~ 0
 LED_G
-Text Label 3800 5650 0    50   ~ 0
+Text Label 3800 5950 0    50   ~ 0
 BTN_R
 Text Label 8450 1100 0    50   ~ 0
@@
 Text Label 3800 4350 0    50   ~ 0
 DPAD_UP
+Text Label 3800 4450 0    50   ~ 0
+DPAD_LEFT
+Text Label 3800 4650 0    50   ~ 0
+DPAD_RIGHT
 Text Label 3800 4550 0    50   ~ 0
-DPAD_LEFT
-Text Label 3800 4450 0    50   ~ 0
-DPAD_RIGHT
-Text Label 3800 4650 0    50   ~ 0
 DPAD_DOWN
 Text Label 6850 1000 2    50   ~ 0
@@
 Text Label 8450 1400 0    50   ~ 0
 BTN_SELECT
-Text Label 3800 5950 0    50   ~ 0
+Text Label 3800 5350 0    50   ~ 0
 BTN_SELECT
 $Sheet
@@
 Text Label 8450 1550 0    50   ~ 0
 BTN_BLUETOOTH
-Text Label 3800 5850 0    50   ~ 0
+Text Label 3800 5450 0    50   ~ 0
 BTN_START
 Text Label 8450 1300 0    50   ~ 0
@@
 Text Label 6850 1800 2    50   ~ 0
 BTN_B
+Text Label 3800 5850 0    50   ~ 0
+BTN_X
 Text Label 3800 5550 0    50   ~ 0
-BTN_X
+BTN_Y
 Text Label 3800 5750 0    50   ~ 0
-BTN_Y
-Text Label 3800 5450 0    50   ~ 0
 BTN_A
-Text Label 3800 5350 0    50   ~ 0
+Text Label 3800 5650 0    50   ~ 0
 BTN_B
 Text Label 6850 4800 2    50   ~ 0
@@
 NoConn ~ 3800 4950
 NoConn ~ 3800 4850
-NoConn ~ 3800 4050
-NoConn ~ 3800 4150
 NoConn ~ 3800 3250
 NoConn ~ 3800 3050
 NoConn ~ 3800 2950
+NoConn ~ 3800 4050
+NoConn ~ 3800 4150
 $EndSCHEMATC
