File: rev-1/rev1/reset.sch (KiCad schematic (older format))
At the start: 7 parts, among them SW14 RESET

Commit message: More work again
Parts:
- C10: value 100n -> 22u
Changed lines of the file:
@@
 P 5150 3700
 F 0 "C10" V 4898 3700 50  0000 C CNN
-F 1 "100n" V 4989 3700 50  0000 C CNN
+F 1 "22u" V 4989 3700 50  0000 C CNN
 F 2 "Capacitor_SMD:C_0603_1608Metric" H 5188 3550 50  0001 C CNN
 F 3 "~" H 5150 3700 50  0001 C CNN
