File: rev-1/rev1/rev1.kicad_pcb (KiCad board)
At the start: 2 copper layers, 145 x 70 mm, 47 parts, among them J1 Conn_01x08_Female, SW1 DPAD_UP, SW10 BTN_Y, SW11 BTN_SELECT, SW12 BTN_A, SW13 BTN_B, SW14 RESET, SW2 BTN_L, SW3 DPAD_DOWN, SW4 BTN_R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

Commit message: More Work, almost done with rev 1
Parts:
- removed the REF** at (178.0, 118.0)
- added REF**: MountingHole_4.3mm_M4, MountingHole:MountingHole_4.3mm_M4, F.Cu at (161.0, 129.0)
- added REF**: MountingHole_4.3mm_M4, MountingHole:MountingHole_4.3mm_M4, F.Cu at (223.0, 118.9)
- added REF**: MountingHole_4.3mm_M4, MountingHole:MountingHole_4.3mm_M4, F.Cu at (99.0, 118.9)
- FID1: value x15y60 -> x15y55
- FID2: value x135y55 -> x135y50
- FID3: value x10y10 -> x10y5
- moved C3 21.4 mm to (150.2, 107.7)
- moved C9 21.4 mm to (151.9, 107.7)
- moved C2 21.4 mm to (145.4, 107.7)
- moved X1 21.3 mm to (147.8, 107.7)
- moved C5 21.3 mm to (143.7, 107.7)
- moved C4 20.9 mm to (146.9, 100.2)
- moved C6 20.2 mm to (145.4, 96.9), turned to 0 degrees
- moved C8 19.8 mm to (146.9, 98.6), turned to 180 degrees
- moved L1 19.0 mm to (141.0, 108.3), turned to 90 degrees
- moved C1 18.8 mm to (141.5, 106.3), turned to 180 degrees
- moved U1 18.6 mm to (141.2, 101.5), turned to 270 degrees
- moved C7 17.0 mm to (142.2, 96.9), turned to 0 degrees
- moved AE1 15.7 mm to (141.0, 123.2)
- moved C11 12.8 mm to (141.5, 122.2), turned to 0 degrees
- moved REF** 3.71 mm to (177.7, 121.7)
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Connections:
- U1 pad 18: /DPAD_RIGHT -> /DPAD_LEFT
- U1 pad 19: /DPAD_LEFT -> /DPAD_DOWN
- U1 pad 20: /DPAD_DOWN -> /DPAD_RIGHT
- U1 pad 37: /BTN_B -> /BTN_SELECT
- U1 pad 38: /BTN_A -> /BTN_START
- U1 pad 39: /BTN_X -> /BTN_Y
- U1 pad 40: /BTN_R -> /BTN_B
- U1 pad 41: /BTN_Y -> /BTN_A
- U1 pad 42: /BTN_START -> /BTN_X
- U1 pad 43: /BTN_SELECT -> /BTN_R
Routing:
- net VCC: track 172.6 -> 110.3 mm
- net /BTN_R: track 88.1 -> 63.4 mm
- net /BTN_Y: track 61.5 -> 44.3 mm
- net /DPAD_DOWN: track 13.3 -> 30.0 mm
- net /BTN_X: track 78.4 -> 62.3 mm
- net /BTN_BLUETOOTH: track 28.3 -> 13.5 mm
- net /SWDCLK: track 53.1 -> 38.6 mm, vias 0 -> 1
- net /P0.18: track 48.9 -> 34.7 mm, vias 0 -> 1
- net /SWDIO: track 58.3 -> 45.1 mm, vias 0 -> 1
- net /BTN_SELECT: track 8.32 -> 21.2 mm
- net /~RESET: track 104.5 -> 116.9 mm
- net /BTN_A: track 88.3 -> 76.9 mm
- net /DPAD_RIGHT: track 5.46 -> 15.8 mm
- net /DPAD_LEFT: track 21.3 -> 30.9 mm
- net /BTN_L: track 33.5 -> 24.8 mm
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Other:
- board size 145 x 70 mm -> 145 x 65 mm
- board text added: "Notes: All mounting holes (both embedded in the pcb and in the milling trace) have a diameter of 4.3mm."

Commit message: More work again
Parts:
- removed the REF** at (161.0, 129.0)
- removed the REF** at (223.0, 118.9)
- removed the REF** at (99.0, 118.9)
- REF** (x2): footprint MountingHole:MountingHole_4.3mm_M4 -> DATX02:MountingHole_4.3mm_M4
Other:
- outline, holes or cut-outs redrawn
- board text added: "R1.250 mm"
- board text added: "R2.150 mm"
- board text removed: "Notes: All mounting holes (both embedded in the pcb and in the milling trace) have a diameter of 4.3mm."
Changed lines of the file:
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@@
   (general
     (thickness 1.6)
-    (drawings 1116)
+    (drawings 1118)
     (tracks 332)
     (zones 0)
-    (modules 49)
+    (modules 46)
     (nets 36)
   )
@@
     (add_net VCC)
   )
-  (module MountingHole:MountingHole_4.3mm_M4 (layer F.Cu)
-    (at 161 128.975)
+  (module DATX02:MountingHole_4.3mm_M4 (layer F.Cu)
+    (at 188.5 93.35)
     (descr "Mounting Hole 4.3mm, no annular, M4")
     (tags "mounting hole 4.3mm no annular m4")
@@
       (effects (font (size 1 1) (thickness 0.15)))
     )
+    (fp_circle (center 0 0) (end 4.55 0) (layer F.CrtYd) (width 0.05))
+    (fp_circle (center 0 0) (end 2.15 0) (layer Cmts.User) (width 0.15))
     (fp_text user %R (at 0.3 0) (layer F.Fab)
       (effects (font (size 1 1) (thickness 0.15)))
     )
-    (fp_circle (center 0 0) (end 4.3 0) (layer Cmts.User) (width 0.15))
-    (fp_circle (center 0 0) (end 4.55 0) (layer F.CrtYd) (width 0.05))
-    (pad "" np_thru_hole circle (at 0 0.025) (size 4.3 4.3) (drill 4.3) (layers *.Cu *.Mask))
-  )
-  (module MountingHole:MountingHole_4.3mm_M4 (layer F.Cu)
-    (at 223 118.9)
+    (pad 1 np_thru_hole circle (at 0 0) (size 4.3 4.3) (drill 4.3) (layers *.Cu *.Mask))
+  )
+  (module DATX02:MountingHole_4.3mm_M4 (layer F.Cu)
+    (at 133.5 93.35)
     (descr "Mounting Hole 4.3mm, no annular, M4")
     (tags "mounting hole 4.3mm no annular m4")
@@
       (effects (font (size 1 1) (thickness 0.15)))
     )
-    (fp_text user %R (at 0.3 0) (layer F.Fab)
-      (effects (font (size 1 1) (thickness 0.15)))
-    )
-    (fp_circle (center 0 0) (end 4.3 0) (layer Cmts.User) (width 0.15))
     (fp_circle (center 0 0) (end 4.55 0) (layer F.CrtYd) (width 0.05))
-    (pad "" np_thru_hole circle (at 0 0) (size 4.3 4.3) (drill 4.3) (layers *.Cu *.Mask))
-  )
-  (module MountingHole:MountingHole_4.3mm_M4 (layer F.Cu)
-    (at 99 118.9)
-    (descr "Mounting Hole 4.3mm, no annular, M4")
-    (tags "mounting hole 4.3mm no annular m4")
-    (attr virtual)
-    (fp_text reference REF** (at 0 -5.3) (layer F.SilkS) hide
-      (effects (font (size 1 1) (thickness 0.15)))
-    )
-    (fp_text value MountingHole_4.3mm_M4 (at 0 5.3) (layer F.Fab)
-      (effects (font (size 1 1) (thickness 0.15)))
-    )
-    (fp_circle (center 0 0) (end 4.55 0) (layer F.CrtYd) (width 0.05))
-    (fp_circle (center 0 0) (end 4.3 0) (layer Cmts.User) (width 0.15))
+    (fp_circle (center 0 0) (end 2.15 0) (layer Cmts.User) (width 0.15))
     (fp_text user %R (at 0.3 0) (layer F.Fab)
       (effects (font (size 1 1) (thickness 0.15)))
@@
     (pad "" smd circle (at 0 0) (size 1 1) (layers F.Cu F.Mask)
       (solder_mask_margin 0.5) (clearance 0.5))
-  )
-  (module MountingHole:MountingHole_4.3mm_M4 (layer F.Cu)
-    (at 188.5 93.35)
-    (descr "Mounting Hole 4.3mm, no annular, M4")
-    (tags "mounting hole 4.3mm no annular m4")
-    (attr virtual)
-    (fp_text reference REF** (at 0 -5.3) (layer F.SilkS) hide
-      (effects (font (size 1 1) (thickness 0.15)))
-    )
-    (fp_text value MountingHole_4.3mm_M4 (at 0 5.3) (layer F.Fab)
-      (effects (font (size 1 1) (thickness 0.15)))
-    )
-    (fp_text user %R (at 0.3 0) (layer F.Fab)
-      (effects (font (size 1 1) (thickness 0.15)))
-    )
-    (fp_circle (center 0 0) (end 4.3 0) (layer Cmts.User) (width 0.15))
-    (fp_circle (center 0 0) (end 4.55 0) (layer F.CrtYd) (width 0.05))
-    (pad 1 np_thru_hole circle (at 0 0) (size 4.3 4.3) (drill 4.3) (layers *.Cu *.Mask))
   )
   (module Diode_SMD:D_0603_1608Metric (layer F.Cu)
@@
       (solder_mask_margin 0.5) (clearance 0.5))
   )
-  (module MountingHole:MountingHole_4.3mm_M4 (layer F.Cu)
-    (at 133.5 93.35)
-    (descr "Mounting Hole 4.3mm, no annular, M4")
-    (tags "mounting hole 4.3mm no annular m4")
-    (attr virtual)
-    (fp_text reference REF** (at 0 -5.3) (layer F.SilkS) hide
-      (effects (font (size 1 1) (thickness 0.15)))
-    )
-    (fp_text value MountingHole_4.3mm_M4 (at 0 5.3) (layer F.Fab)
-      (effects (font (size 1 1) (thickness 0.15)))
-    )
-    (fp_circle (center 0 0) (end 4.55 0) (layer F.CrtYd) (width 0.05))
-    (fp_circle (center 0 0) (end 4.3 0) (layer Cmts.User) (width 0.15))
-    (fp_text user %R (at 0.3 0) (layer F.Fab)
-      (effects (font (size 1 1) (thickness 0.15)))
-    )
-    (pad 1 np_thru_hole circle (at 0 0) (size 4.3 4.3) (drill 4.3) (layers *.Cu *.Mask))
-  )
   (module Capacitor_SMD:C_0402_1005Metric (layer F.Cu)
     (at 141.515 122.25)
@@
     )
   )
-  (gr_line (start 99 116.75) (end 99 121.05) (layer Edge.Cuts) (width 0.2))
-  (gr_text "Notes: \nAll mounting holes (both \nembedded in the pcb and \nin the milling trace) have \na diameter of 4.3mm." (at 57.1 38.7) (layer Cmts.User)
-    (effects (font (size 1.5 1.5) (thickness 0.3)) (justify left))
-  )
+  (gr_text "R1.250 mm" (at 79 105.825) (layer Cmts.User)
+    (effects (font (size 1.4 1.4) (thickness 0.3)))
+  )
+  (gr_line (start 97.725 112.5) (end 78.6 107.325) (layer Cmts.User) (width 0.4))
+  (gr_text "R2.150 mm" (at 80.275 112.325) (layer Cmts.User)
+    (effects (font (size 1.4 1.4) (thickness 0.3)))
+  )
+  (gr_line (start 99 119) (end 79.875 113.825) (layer Cmts.User) (width 0.4))
   (dimension 71.95 (width 0.3) (layer Cmts.User)
     (gr_text "71.950 mm" (at 125.025 49.2) (layer Cmts.User)
@@
   )
   (dimension 134 (width 0.3) (layer Cmts.User)
-    (gr_text "134.000 mm" (at 156 30.5) (layer Cmts.User)
+    (gr_text "134.000 mm" (at 156.004909 31.925) (layer Cmts.User)
       (effects (font (size 1.5 1.5) (thickness 0.3)))
     )
-    (feature1 (pts (xy 223 114) (xy 223 32.013579)))
-    (feature2 (pts (xy 89 114) (xy 89 32.013579)))
-    (crossbar (pts (xy 89 32.6) (xy 223 32.6)))
-    (arrow1a (pts (xy 223 32.6) (xy 221.873496 33.186421)))
-    (arrow1b (pts (xy 223 32.6) (xy 221.873496 32.013579)))
-    (arrow2a (pts (xy 89 32.6) (xy 90.126504 33.186421)))
-    (arrow2b (pts (xy 89 32.6) (xy 90.126504 32.013579)))
+    (feature1 (pts (xy 223.004909 139.013424) (xy 223.004909 33.438579)))
+    (feature2 (pts (xy 89.004909 139.013424) (xy 89.004909 33.438579)))
+    (crossbar (pts (xy 89.004909 34.025) (xy 223.004909 34.025)))
+    (arrow1a (pts (xy 223.004909 34.025) (xy 221.878405 34.611421)))
+    (arrow1b (pts (xy 223.004909 34.025) (xy 221.878405 33.438579)))
+    (arrow2a (pts (xy 89.004909 34.025) (xy 90.131413 34.611421)))
+    (arrow2b (pts (xy 89.004909 34.025) (xy 90.131413 33.438579)))
   )
   (dimension 10 (width 0.3) (layer Cmts.User)
-    (gr_text "10.000 mm" (at 94 65.9) (layer Cmts.User)
+    (gr_text "10.000 mm" (at 94.009898 67.475) (layer Cmts.User)
       (effects (font (size 1.5 1.5) (thickness 0.3)))
     )
-    (feature1 (pts (xy 89 105) (xy 89 67.413579)))
-    (feature2 (pts (xy 99 105) (xy 99 67.413579)))
-    (crossbar (pts (xy 99 68) (xy 89 68)))
-    (arrow1a (pts (xy 89 68) (xy 90.126504 67.413579)))
-    (arrow1b (pts (xy 89 68) (xy 90.126504 68.586421)))
-    (arrow2a (pts (xy 99 68) (xy 97.873496 67.413579)))
-    (arrow2b (pts (xy 99 68) (xy 97.873496 68.586421)))
+    (feature1 (pts (xy 89.009898 139.008305) (xy 89.009898 68.988579)))
+    (feature2 (pts (xy 99.009898 139.008305) (xy 99.009898 68.988579)))
+    (crossbar (pts (xy 99.009898 69.575) (xy 89.009898 69.575)))
+    (arrow1a (pts (xy 89.009898 69.575) (xy 90.136402 68.988579)))
+    (arrow1b (pts (xy 89.009898 69.575) (xy 90.136402 70.161421)))
+    (arrow2a (pts (xy 99.009898 69.575) (xy 97.883394 68.988579)))
+    (arrow2b (pts (xy 99.009898 69.575) (xy 97.883394 70.161421)))
   )
   (gr_arc (start 104 129) (end 104 131.5) (angle 45) (layer Edge.Cuts) (width 0.2))
@@
   (gr_arc (start 133.5 86) (end 133.5 83.5) (angle 90) (layer Edge.Cuts) (width 0.2))
   (gr_arc (start 143.5 86) (end 141 86) (angle 90) (layer Edge.Cuts) (width 0.2))
-  (gr_arc (start 161 129) (end 163.15 129) (angle -180) (layer Dwgs.User) (width 0.2))
+  (gr_arc (start 161 129) (end 163.15 129) (angle -180) (layer Edge.Cuts) (width 0.2))
   (gr_line (start 224.75 125.8) (end 219.8 130.75) (layer Edge.Cuts) (width 0.2))
   (gr_arc (start 218 129) (end 218 131.5) (angle -45) (layer Edge.Cuts) (width 0.2))
@@
   (gr_line (start 143.5 87.5) (end 143.5 86) (layer Edge.Cuts) (width 0.2))
   (gr_line (start 198 86) (end 203 86) (layer Edge.Cuts) (width 0.2))
-  (gr_arc (start 99 118.9) (end 99 121.05) (angle -180) (layer Dwgs.User) (width 0.2))
+  (gr_arc (start 99 118.9) (end 99 121.05) (angle -180) (layer Edge.Cuts) (width 0.2))
   (gr_line (start 178.5 83.5) (end 143.5 83.5) (layer Edge.Cuts) (width 0.2))
   (gr_line (start 143.5 86) (end 178.5 86) (layer Edge.Cuts) (width 0.2))
@@
     (effects (font (size 1.5 1.5) (thickness 0.3)))
   )
-  (gr_arc (start 223 118.9) (end 223 116.75) (angle -180) (layer Dwgs.User) (width 0.2))
+  (gr_arc (start 223 118.9) (end 223 116.75) (angle -180) (layer Edge.Cuts) (width 0.2))
   (gr_text DATX02-19-04 (at 177.85 127.3) (layer F.SilkS)
     (effects (font (size 1.5 1.5) (thickness 0.3)))
@@
   (gr_line (start 203 86) (end 223 106) (layer Edge.Cuts) (width 0.2))
   (gr_line (start 129.4 86) (end 133.5 86) (layer Edge.Cuts) (width 0.2))
-  (gr_line (start 223 124) (end 223 116.75) (layer Edge.Cuts) (width 0.2))
-  (gr_line (start 158.85 129) (end 218 129) (layer Edge.Cuts) (width 0.2))
+  (gr_line (start 223 124) (end 223 121.05) (layer Edge.Cuts) (width 0.2))
+  (gr_line (start 163.15 129) (end 218 129) (layer Edge.Cuts) (width 0.2))
   (gr_line (start 99 124) (end 99 121.05) (layer Edge.Cuts) (width 0.2))
   (gr_line (start 150.5 129) (end 104 129) (layer Edge.Cuts) (width 0.2))
